Commit message: #1 robogardener with one arme

File: robogardener/description/core.xacro (robot description, xacro)
@@ -1,19 +1,20 @@
 <?xml version="1.0"?>
 <robot xmlns:xacro="http://www.ros.org/wiki/xacro" name="robogardener">
+  <xacro:include filename="pantograph.xacro"/>
   <xacro:macro name="robot">
   <!-- constants for robot dimensions-->
   <xacro:property name="PI" value="3.1415926535897931"/>
   <xacro:property name="base_mass" value="6" /> <!-- arbitrary value for base mass -->
-  <xacro:property name="base_width" value="2" />
-  <xacro:property name="base_length" value="5" />
-  <xacro:property name="base_height" value="2" />
-  <xacro:property name="wheel_mass" value="2" /> <!-- arbitrary value for wheel mass -->
-  <xacro:property name="wheel_len" value="1" />
-  <xacro:property name="wheel_radius" value="1" />
-  <link name="odom_link"/>
+  <xacro:property name="base_width" value="0.3" />
+  <xacro:property name="base_length" value="0.2" />
+  <xacro:property name="base_height" value="0.1" />
+  <xacro:property name="wheel_mass" value="0.1" /> <!-- arbitrary value for wheel mass -->
+  <xacro:property name="wheel_len" value="0.05" />
+  <xacro:property name="wheel_radius" value="0.05" />
+  <link name="dummy_link"/>
   <joint name="fixed_base_joint" type="fixed">
-    <parent link="odom_link"/>
+    <parent link="dummy_link"/>
     <child link="base_link"/>
-    <origin xyz="0 0 0" rpy="0 0 0"/>
+    <origin xyz="0 0 0.025" rpy="0 0 0"/>
   </joint>
     <!-- Base Link -->
@@ -41,8 +42,9 @@
       </inertial>
     </link>
-    <joint name="left_wheel_joint" type="continuous">
+    <xacro:pantograph_arm/>
+    <joint name="left_f_wheel_joint" type="continuous">
       <parent link="base_link"/>
-      <child link="left_wheel"/>
-      <origin xyz="0 -${base_length/2} 0" rpy="0 0 0"/>
+      <child link="left_f_wheel"/>
+      <origin xyz="${base_width/4} -${base_length/2} 0" rpy="0 0 0"/>
       <axis xyz="0 1 0"/>
       <dynamics damping="0.2"/>
@@ -50,5 +52,5 @@
     </joint>
     <!-- left wheel Link -->
-    <link name="left_wheel">
+    <link name="left_f_wheel">
       <collision>
         <origin xyz="0 0 0" rpy="${PI/2} 0 0"/>
@@ -73,8 +75,40 @@
         </inertial>
       </link>
-    <joint name="right_wheel_joint" type="continuous">
+      <joint name="left_b_wheel_joint" type="continuous">
       <parent link="base_link"/>
-      <child link="right_wheel"/>
-      <origin xyz="0 ${base_length/2} 0" rpy="0 0 0"/>
+      <child link="left_b_wheel"/>
+      <origin xyz="-${base_width/4} -${base_length/2} 0" rpy="0 0 0"/>
+      <axis xyz="0 1 0"/>
+      <dynamics damping="0.2"/>
+      <limit effort="100" velocity="1.0"/>
+    </joint>
+    <!-- left wheel Link -->
+    <link name="left_b_wheel">
+      <collision>
+        <origin xyz="0 0 0" rpy="${PI/2} 0 0"/>
+        <geometry>
+          <cylinder length="${wheel_len}" radius="${wheel_radius}"/>
+        </geometry>
+      </collision>
+      <visual>
+        <origin xyz="0 0 0" rpy="${PI/2} 0 0"/>
+        <geometry>
+          <cylinder length="${wheel_len}" radius="${wheel_radius}"/>
+        </geometry>
+        <material name="yellow"/>
+      </visual>
+      <inertial>
+        <origin xyz="0 0 0" rpy="${PI/2} 0 0"/>
+        <mass value="${wheel_mass}"/>
+        <inertia
+          ixx="${wheel_mass / 12.0 * (3*wheel_radius*wheel_radius + wheel_len*wheel_len)}" ixy="0.0" ixz="0.0"
+          iyy="${wheel_mass / 12.0 * (3*wheel_radius*wheel_radius + wheel_len*wheel_len)}" iyz="0.0"
+          izz="${wheel_mass / 2.0 * wheel_radius*wheel_radius}"/>
+        </inertial>
+      </link>
+    <joint name="right_f_wheel_joint" type="continuous">
+      <parent link="base_link"/>
+      <child link="right_f_wheel"/>
+      <origin xyz="${base_width/4} ${base_length/2} 0" rpy="0 0 0"/>
       <axis xyz="0 1 0"/>
       <dynamics damping="0.2"/>
@@ -82,5 +116,37 @@
     </joint>
     <!-- right wheel Link -->
-    <link name="right_wheel">
+    <link name="right_f_wheel">
+      <collision>
+        <origin xyz="0 0 0" rpy="${PI/2} 0 0"/>
+        <geometry>
+          <cylinder length="${wheel_len}" radius="${wheel_radius}"/>
+        </geometry>
+      </collision>
+      <visual>
+        <origin xyz="0 0 0" rpy="${PI/2} 0 0"/>
+        <geometry>
+          <cylinder length="${wheel_len}" radius="${wheel_radius}"/>
+        </geometry>
+        <material name="yellow"/>
+      </visual>
+      <inertial>
+        <origin xyz="0 0 0" rpy="${PI/2} 0 0"/>
+        <mass value="${wheel_mass}"/>
+        <inertia
+          ixx="${wheel_mass / 12.0 * (3*wheel_radius*wheel_radius + wheel_len*wheel_len)}" ixy="0.0" ixz="0.0"
+          iyy="${wheel_mass / 12.0 * (3*wheel_radius*wheel_radius + wheel_len*wheel_len)}" iyz="0.0"
+          izz="${wheel_mass / 2.0 * wheel_radius*wheel_radius}"/>
+        </inertial>
+      </link>
+    <joint name="right_b_wheel_joint" type="continuous">
+      <parent link="base_link"/>
+      <child link="right_b_wheel"/>
+      <origin xyz="-${base_width/4} ${base_length/2} 0" rpy="0 0 0"/>
+      <axis xyz="0 1 0"/>
+      <dynamics damping="0.2"/>
+      <limit effort="100" velocity="1.0"/>
+    </joint>
+    <!-- right wheel Link -->
+    <link name="right_b_wheel">
       <collision>
         <origin xyz="0 0 0" rpy="${PI/2} 0 0"/>

File: robogardener/description/gz_control.xacro (robot description, xacro)
@@ -18,27 +18,42 @@
         </joint>
     </ros2_control-->
+    <!-- constants for robot dimensions-->
+  <xacro:property name="PI" value="3.1415926535897931"/>
+  <xacro:property name="base_mass" value="6" /> <!-- arbitrary value for base mass -->
+  <xacro:property name="base_width" value="0.3" />
+  <xacro:property name="base_length" value="0.2" />
+  <xacro:property name="base_height" value="0.1" />
+  <xacro:property name="wheel_mass" value="0.1" /> <!-- arbitrary value for wheel mass -->
+  <xacro:property name="wheel_len" value="0.05" />
+  <xacro:property name="wheel_radius" value="0.05" />
     <gazebo>
         <plugin name="gz::sim::systems::DiffDrive" filename="gz-sim-diff-drive-system">
-            <!-- Wheel Information -->
-            <left_joint>left_wheel_joint</left_joint>
-            <right_joint>right_wheel_joint</right_joint>
-            <wheel_separation>5</wheel_separation>
-            <wheel_radius>1</wheel_radius>
-            <!-- Input -->
-            <topic>/cmd_vel</topic>
-            <!-- Output -->
-            <frame_id>odom</frame_id>
-            <child_frame_id>base_link</child_frame_id>
-            <odom_topic>odom</odom_topic>
-            <odom_publish_frequency>50</odom_publish_frequency>
-            <!-- TF Publishing -->
-            <publish_tf>true</publish_tf>
-        </plugin>
+            <!-- Left wheels -->
+      <left_joint>left_f_wheel_joint</left_joint>
+      <left_joint>left_b_wheel_joint</left_joint>
+      <!-- Right wheels -->
+      <right_joint>right_f_wheel_joint</right_joint>
+      <right_joint>right_b_wheel_joint</right_joint>
+      <!-- Wheel geometry -->
+      <wheel_separation>${base_length}</wheel_separation>  <!-- consider using actual separation -->
+      <wheel_radius>${wheel_radius}</wheel_radius>
+      <!-- Topics -->
+      <topic>/cmd_vel</topic>
+      <odom_topic>odom</odom_topic>
+      <!-- Frames -->
+      <frame_id>odom</frame_id>
+      <child_frame_id>base_link</child_frame_id>
+      <!-- Publish settings -->
+      <odom_publish_frequency>50</odom_publish_frequency>
+      <publish_tf>true</publish_tf>
+    </plugin>
         <plugin filename="gz-sim-joint-state-publisher-system"
             name="gz::sim::systems::JointStatePublisher">
             <topic>joint_states</topic>
-            <joint_name>left_wheel_joint</joint_name>
-            <joint_name>right_wheel_joint</joint_name>
-        </plugin>
-    </gazebo>
+      <joint_name>left_f_wheel_joint</joint_name>
+      <joint_name>left_b_wheel_joint</joint_name>
+      <joint_name>right_f_wheel_joint</joint_name>
+      <joint_name>right_b_wheel_joint</joint_name>
+    </plugin>
+  </gazebo>
 </robot>

File: robogardener/description/materials.xacro (robot description, xacro)
@@ -17,3 +17,6 @@
     <color rgba="0.8 0.0 0.0 1.0"/>
   </material>
+  <material name="green">
+  <color rgba="0.0 1.0 0.0 1.0"/>
+  </material>
 </robot>

Commit message: #3

File: robogardener/description/core.xacro (robot description, xacro)
@@ -1,6 +1,4 @@
 <?xml version="1.0"?>
-<robot xmlns:xacro="http://www.ros.org/wiki/xacro" name="robogardener">
-  <xacro:include filename="pantograph.xacro"/>
-  <xacro:macro name="robot">
+<robot xmlns:xacro="http://www.ros.org/wiki/xacro" >
   <!-- constants for robot dimensions-->
   <xacro:property name="PI" value="3.1415926535897931"/>
@@ -12,10 +10,4 @@
   <xacro:property name="wheel_len" value="0.05" />
   <xacro:property name="wheel_radius" value="0.05" />
-  <link name="dummy_link"/>
-  <joint name="fixed_base_joint" type="fixed">
-    <parent link="dummy_link"/>
-    <child link="base_link"/>
-    <origin xyz="0 0 0.025" rpy="0 0 0"/>
-  </joint>
     <!-- Base Link -->
   <link name="base_link">
@@ -171,4 +163,3 @@
         </inertial>
       </link>
-  </xacro:macro>
 </robot>

File: robogardener/description/gz_control.xacro (robot description, xacro)
@@ -1,8 +1,4 @@
 <?xml version="1.0"?>
 <robot xmlns:xacro="http://www.ros.org/wiki/xacro">
-    <ros2_control name="robogardener_controller" type="system">
-    <hardware>
-        <plugin>gz_ros2_control/GazeboSystem</plugin>
-    </hardware>
     <joint name="left_f_wheel_joint">
         <command_interface name="velocity"/>
@@ -25,4 +21,3 @@
         <state_interface name="velocity"/>
     </joint>
-    </ros2_control>
 </robot>

File: robogardener/description/robo.urdf.xacro (robot description, xacro)
@@ -1,15 +1,13 @@
 <?xml version="1.0"?>
 <robot xmlns:xacro="http://www.ros.org/wiki/xacro" name="robogardener">
-    <!-- Arguments -->
-    <xacro:arg name="sim_mode" default="true" />
-    <!-- Includes -->
-    <xacro:include filename="core.xacro" />
-    <xacro:include filename="materials.xacro" />
-    <xacro:include filename="gz_control.xacro" />
-    <xacro:include filename="ros2_control.xacro" />
-    <gazebo>
-        <plugin filename="libgz_ros2_control-system.so" name="gz_ros2_control::GazeboSystemPlugin"/>
-    </gazebo>
-    <!-- Macro Invocation -->
-    <xacro:robot />
+  <xacro:arg name="prefix" default="" />
+  <xacro:arg name="use_mock_hardware" default="false" />
+  <xacro:include filename="core.xacro" />
+  <xacro:include filename="materials.xacro" />
+  <xacro:include filename="ros2_control.xacro" />
+  <!-- Actually call the ros2_control macro -->
+  <xacro:robogardener_ros2_control
+    name="robogardener"
+    prefix="$(arg prefix)"
+    use_mock_hardware="$(arg use_mock_hardware)"/>
 </robot>

File: robogardener/description/ros2_control.xacro (robot description, xacro)
@@ -1,34 +1,40 @@
 <?xml version="1.0"?>
 <robot xmlns:xacro="http://www.ros.org/wiki/xacro">
-  <!-- ROS2 Control Integration -->
-  <ros2_control name="controller_manager" type="system">
-    <hardware>
-      <!-- Gazebo plugin -->
-      <plugin>gz_ros2_control/GazeboSystem</plugin>
-    </hardware>
-    <!-- Left front wheel -->
-    <joint name="left_f_wheel_joint">
-      <command_interface name="velocity"/>
-      <state_interface name="position"/>
-      <state_interface name="velocity"/>
-    </joint>
-    <!-- Left back wheel -->
-    <joint name="left_b_wheel_joint">
-      <command_interface name="velocity"/>
-      <state_interface name="position"/>
-      <state_interface name="velocity"/>
-    </joint>
-    <!-- Right front wheel -->
-    <joint name="right_f_wheel_joint">
-      <command_interface name="velocity"/>
-      <state_interface name="position"/>
-      <state_interface name="velocity"/>
-    </joint>
-    <!-- Right back wheel -->
-    <joint name="right_b_wheel_joint">
-      <command_interface name="velocity"/>
-      <state_interface name="position"/>
-      <state_interface name="velocity"/>
-    </joint>
-  </ros2_control>
+  <xacro:macro name="robogardener_ros2_control" params="name prefix use_mock_hardware">
+    <ros2_control name="${name}" type="system">
+      <xacro:unless value="${use_mock_hardware}">
+        <hardware>
+          <plugin>gz_ros2_control/GazeboSystem</plugin>
+          <param name="robot_description">{load_urdf('$(find robogardener)/urdf/robo.urdf.xacro')}</param>
+        </hardware>
+      </xacro:unless>
+      <xacro:if value="${use_mock_hardware}">
+        <hardware>
+          <plugin>mock_components/GenericSystem</plugin>
+          <param name="state_interfaces">position,velocity</param>
+          <param name="command_interfaces">velocity</param>
+        </hardware>
+      </xacro:if>
+      <joint name="${prefix}left_f_wheel_joint">
+        <command_interface name="velocity"/>
+        <state_interface name="position"/>
+        <state_interface name="velocity"/>
+      </joint>
+      <joint name="${prefix}left_b_wheel_joint">
+        <command_interface name="velocity"/>
+        <state_interface name="position"/>
+        <state_interface name="velocity"/>
+      </joint>
+      <joint name="${prefix}right_f_wheel_joint">
+        <command_interface name="velocity"/>
+        <state_interface name="position"/>
+        <state_interface name="velocity"/>
+      </joint>
+      <joint name="${prefix}right_b_wheel_joint">
+        <command_interface name="velocity"/>
+        <state_interface name="position"/>
+        <state_interface name="velocity"/>
+      </joint>
+    </ros2_control>
+  </xacro:macro>
 </robot>
