Commit message: #3

File: robogardener/description/core.xacro (robot description, xacro)
@@ -1,165 +1,204 @@
 <?xml version="1.0"?>
-<robot xmlns:xacro="http://www.ros.org/wiki/xacro" >
-  <!-- constants for robot dimensions-->
+<robot name="robogardener" xmlns:xacro="http://www.ros.org/wiki/xacro">
+  <!-- Constants -->
   <xacro:property name="PI" value="3.1415926535897931"/>
-  <xacro:property name="base_mass" value="6" /> <!-- arbitrary value for base mass -->
-  <xacro:property name="base_width" value="0.3" />
-  <xacro:property name="base_length" value="0.2" />
-  <xacro:property name="base_height" value="0.1" />
-  <xacro:property name="wheel_mass" value="0.1" /> <!-- arbitrary value for wheel mass -->
-  <xacro:property name="wheel_len" value="0.05" />
-  <xacro:property name="wheel_radius" value="0.05" />
-    <!-- Base Link -->
+  <!-- Physical dimensions (converted to meters) -->
+  <xacro:property name="wheel_width" value="0.055" />  <!-- 5.5cm -->
+  <xacro:property name="wheel_radius" value="0.0575" /> <!-- 11.5cm diameter -->
+  <!-- Wheel positions -->
+  <xacro:property name="wheelbase_x" value="0.215" /> <!-- 21.5cm front-to-back -->
+  <xacro:property name="wheelbase_y" value="0.195" /> <!-- 19.5cm left-to-right -->
+  <!-- Chassis dimensions -->
+  <xacro:property name="chassis_length" value="0.37" /> <!-- 37cm -->
+  <xacro:property name="chassis_width" value="0.195" /> <!-- 19.5cm -->
+  <xacro:property name="chassis_height" value="0.03" /> <!-- 3cm -->
+  <xacro:property name="base_height" value="0.06" /> <!-- 6cm rod height -->
+  <!-- Mass properties (estimated) -->
+  <xacro:property name="chassis_mass" value="2.0" /> <!-- kg -->
+  <xacro:property name="wheel_mass" value="0.3" /> <!-- kg -->
+  <link name="odom">
+    <inertial>
+      <mass value="0.001"/>
+      <inertia ixx="0.001" ixy="0" ixz="0" iyy="0.001" iyz="0" izz="0.001"/>
+    </inertial>
+  </link>
+  <joint name="odom_joint" type="floating">
+    <parent link="odom"/>
+    <child link="base_link"/>
+  </joint>
+  <!-- Main chassis link -->
   <link name="base_link">
-    <collision>
-      <origin xyz="0 0 0" rpy="0 0 0"/>
-      <geometry>
-        <box size="${base_width} ${base_length} ${base_height}"/>
-      </geometry>
-    </collision>
     <visual>
       <origin xyz="0 0 ${base_height/2}" rpy="0 0 0"/>
       <geometry>
-        <box size="${base_width} ${base_length} ${base_height}"/>
-      </geometry>
-      <material name="white"/>
-    </visual>
-    <inertial>
-      <origin xyz="0 0 0" rpy="0 0 0"/>
-      <mass value="${base_mass}"/>
-      <inertia
-        ixx="${base_mass / 12.0 * (base_length*base_length + base_height*base_height)}" ixy="0.0" ixz="0.0"
-        iyy="${base_mass / 12.0 * (base_height*base_height + base_width*base_width)}" iyz="0.0"
-        izz="${base_mass / 12.0 * (base_width*base_width + base_length*base_length)}"/>
-      </inertial>
-    </link>
-    <!--xacro:pantograph_arm/ -->
-    <joint name="left_f_wheel_joint" type="continuous">
-      <parent link="base_link"/>
-      <child link="left_f_wheel"/>
-      <origin xyz="${base_width/4} -${base_length/2} 0" rpy="0 0 0"/>
-      <axis xyz="0 1 0"/>
-      <dynamics damping="0.2"/>
-      <limit effort="100" velocity="1.0"/>
+        <box size="${chassis_length} ${chassis_width} ${chassis_height}"/>
+      </geometry>
+      <material name="black"/>
+    </visual>
+    <collision>
+      <origin xyz="0 0 ${base_height/2}" rpy="0 0 0"/>
+      <geometry>
+        <box size="${chassis_length} ${chassis_width} ${chassis_height}"/>
+      </geometry>
+    </collision>
+    <inertial>
+      <origin xyz="0 0 ${base_height/2}"/>
+      <mass value="${chassis_mass}"/>
+      <inertia
+        ixx="${chassis_mass/12 * (chassis_width*chassis_width + chassis_height*chassis_height)}" ixy="0" ixz="0"
+        iyy="${chassis_mass/12 * (chassis_length*chassis_length + chassis_height*chassis_height)}" iyz="0"
+        izz="${chassis_mass/12 * (chassis_length*chassis_length + chassis_width*chassis_width)}"/>
+    </inertial>
+  </link>
+  <!-- All wheels are FIXED to chassis (mechanically linked) -->
+  <!-- Front Left Wheel -->
+  <link name="left_f_wheel">
+    <visual>
+      <origin xyz="0 0 0" rpy="${PI/2} 0 0"/>
+      <geometry>
+        <cylinder radius="${wheel_radius}" length="${wheel_width}"/>
+      </geometry>
+      <material name="yellow"/>
+    </visual>
+    <collision>
+      <origin xyz="0 0 0" rpy="${PI/2} 0 0"/>
+      <geometry>
+        <cylinder radius="${wheel_radius}" length="${wheel_width}"/>
+      </geometry>
+    </collision>
+    <inertial>
+      <origin xyz="0 0 0" rpy="${PI/2} 0 0"/>
+      <mass value="${wheel_mass}"/>
+      <inertia
+        ixx="${wheel_mass/12 * (3*wheel_radius*wheel_radius + wheel_width*wheel_width)}" ixy="0" ixz="0"
+        iyy="${wheel_mass/12 * (3*wheel_radius*wheel_radius + wheel_width*wheel_width)}" iyz="0"
+        izz="${wheel_mass/2 * wheel_radius*wheel_radius}"/>
+    </inertial>
+  </link>
+  <joint name="left_f_wheel_joint" type="fixed">
+    <parent link="base_link"/>
+    <child link="left_f_wheel"/>
+    <origin xyz="${wheelbase_x/2} ${-wheelbase_y/2} 0" rpy="0 0 0"/>
+  </joint>
+  <!-- Front Right Wheel (mirror of left) -->
+  <link name="right_f_wheel">
+    <!-- Same visual/collision/inertial as left wheel -->
+    <visual>
+      <origin xyz="0 0 0" rpy="${PI/2} 0 0"/>
+      <geometry>
+        <cylinder radius="${wheel_radius}" length="${wheel_width}"/>
+      </geometry>
+      <material name="yellow"/>
+    </visual>
+    <collision>
+      <origin xyz="0 0 0" rpy="${PI/2} 0 0"/>
+      <geometry>
+        <cylinder radius="${wheel_radius}" length="${wheel_width}"/>
+      </geometry>
+    </collision>
+    <inertial>
+      <origin xyz="0 0 0" rpy="${PI/2} 0 0"/>
+      <mass value="${wheel_mass}"/>
+      <inertia
+        ixx="${wheel_mass/12 * (3*wheel_radius*wheel_radius + wheel_width*wheel_width)}" ixy="0" ixz="0"
+        iyy="${wheel_mass/12 * (3*wheel_radius*wheel_radius + wheel_width*wheel_width)}" iyz="0"
+        izz="${wheel_mass/2 * wheel_radius*wheel_radius}"/>
+    </inertial>
+  </link>
+  <joint name="right_f_wheel_joint" type="fixed">
+    <parent link="base_link"/>
+    <child link="right_f_wheel"/>
+    <origin xyz="${wheelbase_x/2} ${wheelbase_y/2} 0" rpy="0 0 0"/>
+  </joint>
+  <!-- Rear Wheels (same as front but negative x position) -->
+  <link name="left_b_wheel">
+    <visual>
+      <origin xyz="0 0 0" rpy="${PI/2} 0 0"/>
+      <geometry>
+        <cylinder radius="${wheel_radius}" length="${wheel_width}"/>
+      </geometry>
+      <material name="blue"/>
+    </visual>
+    <collision>
+      <origin xyz="0 0 0" rpy="${PI/2} 0 0"/>
+      <geometry>
+        <cylinder radius="${wheel_radius}" length="${wheel_width}"/>
+      </geometry>
+    </collision>
+    <inertial>
+      <origin xyz="0 0 0" rpy="${PI/2} 0 0"/>
+      <mass value="${wheel_mass}"/>
+      <inertia
+        ixx="${wheel_mass/12 * (3*wheel_radius*wheel_radius + wheel_width*wheel_width)}" ixy="0" ixz="0"
+        iyy="${wheel_mass/12 * (3*wheel_radius*wheel_radius + wheel_width*wheel_width)}" iyz="0"
+        izz="${wheel_mass/2 * wheel_radius*wheel_radius}"/>
+    </inertial>
+  </link>
+  <joint name="left_b_wheel_joint" type="fixed">
+    <parent link="base_link"/>
+    <child link="left_b_wheel"/>
+    <origin xyz="${-wheelbase_x/2} ${-wheelbase_y/2} 0" rpy="0 0 0"/>
+  </joint>
+  <link name="right_b_wheel">
+    <visual>
+      <origin xyz="0 0 0" rpy="${PI/2} 0 0"/>
+      <geometry>
+        <cylinder radius="${wheel_radius}" length="${wheel_width}"/>
+      </geometry>
+      <material name="blue"/>
+    </visual>
+    <collision>
+      <origin xyz="0 0 0" rpy="${PI/2} 0 0"/>
+      <geometry>
+        <cylinder radius="${wheel_radius}" length="${wheel_width}"/>
+      </geometry>
+    </collision>
+    <inertial>
+      <origin xyz="0 0 0" rpy="${PI/2} 0 0"/>
+      <mass value="${wheel_mass}"/>
+      <inertia
+        ixx="${wheel_mass/12 * (3*wheel_radius*wheel_radius + wheel_width*wheel_width)}" ixy="0" ixz="0"
+        iyy="${wheel_mass/12 * (3*wheel_radius*wheel_radius + wheel_width*wheel_width)}" iyz="0"
+        izz="${wheel_mass/2 * wheel_radius*wheel_radius}"/>
+    </inertial>
+  </link>
+  <joint name="right_b_wheel_joint" type="fixed">
+    <parent link="base_link"/>
+    <child link="right_b_wheel"/>
+    <origin xyz="${-wheelbase_x/2} ${wheelbase_y/2} 0" rpy="0 0 0"/>
+  </joint>
+  <!-- Virtual drive joint for the single motor -->
+  <link name="virtual_drive_link">
+    <inertial>
+      <mass value="0.001"/>
+      <inertia ixx="0.001" ixy="0" ixz="0" iyy="0.001" iyz="0" izz="0.001"/>
+    </inertial>
+  </link>
+  <joint name="main_drive_joint" type="continuous">
+    <parent link="base_link"/>
+    <child link="virtual_drive_link"/>
+    <axis xyz="0 1 0"/>
+  </joint>
+  <ros2_control name="SingleMotorDrive" type="system">
+    <hardware>
+      <plugin>ros2_control_gz/Ros2ControlGazeboSystem</plugin>
+    </hardware>
+    <joint name="main_drive_joint">
+      <command_interface name="velocity"/>
+      <state_interface name="position"/>
+      <state_interface name="velocity"/>
     </joint>
-    <!-- left wheel Link -->
-    <link name="left_f_wheel">
-      <collision>
-        <origin xyz="0 0 0" rpy="${PI/2} 0 0"/>
-        <geometry>
-          <cylinder length="${wheel_len}" radius="${wheel_radius}"/>
-        </geometry>
-      </collision>
-      <visual>
-        <origin xyz="0 0 0" rpy="${PI/2} 0 0"/>
-        <geometry>
-          <cylinder length="${wheel_len}" radius="${wheel_radius}"/>
-        </geometry>
-        <material name="yellow"/>
-      </visual>
-      <inertial>
-        <origin xyz="0 0 0" rpy="${PI/2} 0 0"/>
-        <mass value="${wheel_mass}"/>
-        <inertia
-          ixx="${wheel_mass / 12.0 * (3*wheel_radius*wheel_radius + wheel_len*wheel_len)}" ixy="0.0" ixz="0.0"
-          iyy="${wheel_mass / 12.0 * (3*wheel_radius*wheel_radius + wheel_len*wheel_len)}" iyz="0.0"
-          izz="${wheel_mass / 2.0 * wheel_radius*wheel_radius}"/>
-        </inertial>
-      </link>
-      <joint name="left_b_wheel_joint" type="continuous">
-      <parent link="base_link"/>
-      <child link="left_b_wheel"/>
-      <origin xyz="-${base_width/4} -${base_length/2} 0" rpy="0 0 0"/>
-      <axis xyz="0 1 0"/>
-      <dynamics damping="0.2"/>
-      <limit effort="100" velocity="1.0"/>
-    </joint>
-    <!-- left wheel Link -->
-    <link name="left_b_wheel">
-      <collision>
-        <origin xyz="0 0 0" rpy="${PI/2} 0 0"/>
-        <geometry>
-          <cylinder length="${wheel_len}" radius="${wheel_radius}"/>
-        </geometry>
-      </collision>
-      <visual>
-        <origin xyz="0 0 0" rpy="${PI/2} 0 0"/>
-        <geometry>
-          <cylinder length="${wheel_len}" radius="${wheel_radius}"/>
-        </geometry>
-        <material name="yellow"/>
-      </visual>
-      <inertial>
-        <origin xyz="0 0 0" rpy="${PI/2} 0 0"/>
-        <mass value="${wheel_mass}"/>
-        <inertia
-          ixx="${wheel_mass / 12.0 * (3*wheel_radius*wheel_radius + wheel_len*wheel_len)}" ixy="0.0" ixz="0.0"
-          iyy="${wheel_mass / 12.0 * (3*wheel_radius*wheel_radius + wheel_len*wheel_len)}" iyz="0.0"
-          izz="${wheel_mass / 2.0 * wheel_radius*wheel_radius}"/>
-        </inertial>
-      </link>
-    <joint name="right_f_wheel_joint" type="continuous">
-      <parent link="base_link"/>
-      <child link="right_f_wheel"/>
-      <origin xyz="${base_width/4} ${base_length/2} 0" rpy="0 0 0"/>
-      <axis xyz="0 1 0"/>
-      <dynamics damping="0.2"/>
-      <limit effort="100" velocity="1.0"/>
-    </joint>
-    <!-- right wheel Link -->
-    <link name="right_f_wheel">
-      <collision>
-        <origin xyz="0 0 0" rpy="${PI/2} 0 0"/>
-        <geometry>
-          <cylinder length="${wheel_len}" radius="${wheel_radius}"/>
-        </geometry>
-      </collision>
-      <visual>
-        <origin xyz="0 0 0" rpy="${PI/2} 0 0"/>
-        <geometry>
-          <cylinder length="${wheel_len}" radius="${wheel_radius}"/>
-        </geometry>
-        <material name="yellow"/>
-      </visual>
-      <inertial>
-        <origin xyz="0 0 0" rpy="${PI/2} 0 0"/>
-        <mass value="${wheel_mass}"/>
-        <inertia
-          ixx="${wheel_mass / 12.0 * (3*wheel_radius*wheel_radius + wheel_len*wheel_len)}" ixy="0.0" ixz="0.0"
-          iyy="${wheel_mass / 12.0 * (3*wheel_radius*wheel_radius + wheel_len*wheel_len)}" iyz="0.0"
-          izz="${wheel_mass / 2.0 * wheel_radius*wheel_radius}"/>
-        </inertial>
-      </link>
-    <joint name="right_b_wheel_joint" type="continuous">
-      <parent link="base_link"/>
-      <child link="right_b_wheel"/>
-      <origin xyz="-${base_width/4} ${base_length/2} 0" rpy="0 0 0"/>
-      <axis xyz="0 1 0"/>
-      <dynamics damping="0.2"/>
-      <limit effort="100" velocity="1.0"/>
-    </joint>
-    <!-- right wheel Link -->
-    <link name="right_b_wheel">
-      <collision>
-        <origin xyz="0 0 0" rpy="${PI/2} 0 0"/>
-        <geometry>
-          <cylinder length="${wheel_len}" radius="${wheel_radius}"/>
-        </geometry>
-      </collision>
-      <visual>
-        <origin xyz="0 0 0" rpy="${PI/2} 0 0"/>
-        <geometry>
-          <cylinder length="${wheel_len}" radius="${wheel_radius}"/>
-        </geometry>
-        <material name="yellow"/>
-      </visual>
-      <inertial>
-        <origin xyz="0 0 0" rpy="${PI/2} 0 0"/>
-        <mass value="${wheel_mass}"/>
-        <inertia
-          ixx="${wheel_mass / 12.0 * (3*wheel_radius*wheel_radius + wheel_len*wheel_len)}" ixy="0.0" ixz="0.0"
-          iyy="${wheel_mass / 12.0 * (3*wheel_radius*wheel_radius + wheel_len*wheel_len)}" iyz="0.0"
-          izz="${wheel_mass / 2.0 * wheel_radius*wheel_radius}"/>
-        </inertial>
-      </link>
+  </ros2_control>
+  <gazebo>
+    <plugin filename="libgazebo_ros_diff_drive.so" name="diff_drive">
+      <command_topic>cmd_vel</command_topic>
+      <odometry_topic>odom</odometry_topic>
+      <odometry_frame>odom</odometry_frame>
+      <robot_base_frame>base_link</robot_base_frame>
+      <wheel_separation>${wheelbase_y}</wheel_separation> <!-- Distance between wheels -->
+      <wheel_diameter>${2*wheel_radius}</wheel_diameter>
+      <publish_odom>true</publish_odom>
+      <publish_odom_tf>true</publish_odom_tf>
+    </plugin>
+  </gazebo>
 </robot>

File: robogardener/description/robo.urdf.xacro (robot description, xacro)
@@ -1,13 +1,13 @@
 <?xml version="1.0"?>
 <robot xmlns:xacro="http://www.ros.org/wiki/xacro" name="robogardener">
-  <xacro:arg name="prefix" default="" />
   <xacro:arg name="use_mock_hardware" default="false" />
+  <!-- Includes -->
   <xacro:include filename="core.xacro" />
   <xacro:include filename="materials.xacro" />
-  <xacro:include filename="ros2_control.xacro" />
-  <!-- Actually call the ros2_control macro -->
+  <xacro:include filename="$(find robogardener)/description/ros2_control.xacro" />
+  <!-- Call macro -->
   <xacro:robogardener_ros2_control
     name="robogardener"
-    prefix="$(arg prefix)"
+    prefix=""
     use_mock_hardware="$(arg use_mock_hardware)"/>
 </robot>

File: robogardener/description/ros2_control.xacro (robot description, xacro)
@@ -3,33 +3,13 @@
   <xacro:macro name="robogardener_ros2_control" params="name prefix use_mock_hardware">
     <ros2_control name="${name}" type="system">
-      <xacro:unless value="${use_mock_hardware}">
-        <hardware>
-          <plugin>gz_ros2_control/GazeboSystem</plugin>
-          <param name="robot_description">{load_urdf('$(find robogardener)/urdf/robo.urdf.xacro')}</param>
-        </hardware>
-      </xacro:unless>
       <xacro:if value="${use_mock_hardware}">
         <hardware>
           <plugin>mock_components/GenericSystem</plugin>
-          <param name="state_interfaces">position,velocity</param>
+          <param name="joints">main_drive_joint</param>
           <param name="command_interfaces">velocity</param>
+          <param name="state_interfaces">position, velocity</param>
         </hardware>
       </xacro:if>
-      <joint name="${prefix}left_f_wheel_joint">
-        <command_interface name="velocity"/>
-        <state_interface name="position"/>
-        <state_interface name="velocity"/>
-      </joint>
-      <joint name="${prefix}left_b_wheel_joint">
-        <command_interface name="velocity"/>
-        <state_interface name="position"/>
-        <state_interface name="velocity"/>
-      </joint>
-      <joint name="${prefix}right_f_wheel_joint">
-        <command_interface name="velocity"/>
-        <state_interface name="position"/>
-        <state_interface name="velocity"/>
-      </joint>
-      <joint name="${prefix}right_b_wheel_joint">
+      <joint name="main_drive_joint">
         <command_interface name="velocity"/>
         <state_interface name="position"/>

File: robogardener/description/temp.urdf (robot description, URDF)
Before this commit: robot robogardener, 5 links, 4 joints
Links:
- added link virtual_drive_link
- link base_link: mass 6 -> 2.0; geometry collision box size=0.37 0.195 0.03; visual box size=0.37 0.195 0.03
- link left_b_wheel: mass 0.1 -> None; geometry 
- link left_f_wheel: mass 0.1 -> 0.3; geometry collision cylinder length=0.055 radius=0.0575; visual cylinder length=0.055 radius=0.0575
- link right_b_wheel: mass 0.1 -> None; geometry 
- link right_f_wheel: mass 0.1 -> None; geometry visual cylinder length=0.055 radius=0.0575
Joints:
- added joint main_drive_joint: type continuous, parent base_link, child virtual_drive_link, axis 0 1 0, limit effort=100 velocity=10.0
- joint left_b_wheel_joint: axis 0.707 0.707 0 -> (none); limit effort=100 velocity=1.0 -> (none); origin xyz=-0.075 -0.1 0 rpy=0 0 0 -> xyz=-0.1075 -0.0975 0 rpy=0 0 0; type continuous -> fixed
- joint left_f_wheel_joint: axis 0 1 0 -> (none); limit effort=100 velocity=1.0 -> (none); origin xyz=0.075 -0.1 0 rpy=0 0 0 -> xyz=0.1075 -0.0975 0 rpy=0 0 0; type continuous -> fixed
- joint right_b_wheel_joint: axis 0.707 0.707 0 -> (none); limit effort=100 velocity=1.0 -> (none); origin xyz=-0.075 0.1 0 rpy=0 0 0 -> xyz=-0.1075 0.0975 0 rpy=0 0 0; type continuous -> fixed
- joint right_f_wheel_joint: axis 0.707 0.707 0 -> (none); limit effort=100 velocity=1.0 -> (none); origin xyz=0.075 0.1 0 rpy=0 0 0 -> xyz=0.1075 0.0975 0 rpy=0 0 0; type continuous -> fixed
